Commit message: Fase 1 empezada

File: P1/barrera.urdf (robot description, URDF)
Before this commit: robot rampa, 3 links, 2 joints
Links:
- link rampa_derecha: mass 100.0 -> 10.0
- link rampa_izquierda: mass 100.0 -> 10.0

Commit message: Fase 1 terminada

File: P1/barrera.urdf (robot description, URDF)
Before this commit: robot rampa, 3 links, 2 joints
Links:
- removed link base_link
- removed link rampa_derecha
- removed link rampa_izquierda
- added link barrier_link, mass 5.0; collision box size=2 0.1 0.1; visual box size=2 0.1 0.1
- added link post_link, mass 200; collision cylinder length=1 radius=0.1; visual cylinder length=1 radius=0.1
Joints:
- removed joint rampa_derecha_joint
- removed joint rampa_izquierda_joint
- added joint barrier_joint: type revolute, parent post_link, child barrier_link, origin xyz=0 0.75 -0.25 rpy=0 0 0, axis 0 0 1, limit lower=-3.14 upper=3.14 effort=1000 velocity=10

File: P1/plataforma.urdf (robot description, URDF)
Before this commit: robot plataforma, 1 links, 0 joints
Links:
- removed link plataforma_link
- added link platform_link, mass 100.0; collision box size=3 1 0.05; visual box size=3 1 0.05

File: P1/rampa.urdf (robot description, URDF)
Before this commit: robot rampa, 3 links, 2 joints
Links:
- removed link rampa_derecha
- removed link rampa_izquierda
- added link ramp_left_link, mass 100.0; collision box size=2 3.16 0.01; visual box size=2 3.16 0.01
- added link ramp_right_link, mass 100.0; collision box size=2 3.16 0.01; visual box size=2 3.16 0.01
Joints:
- removed joint rampa_derecha_joint
- removed joint rampa_izquierda_joint
- added joint ramp_left_joint: type fixed, parent base_link, child ramp_left_link, origin xyz=0 3.5 0 rpy=0 0 0
- added joint ramp_right_joint: type fixed, parent base_link, child ramp_right_link, origin xyz=0 -3.5 0 rpy=0 0 0

Commit message: Fase 3 terminada

File: P1/barrera.urdf (robot description, URDF)
Before this commit: robot barrier, 2 links, 1 joints
Links:
- link barrier_link: geometry collision cylinder length=2 radius=0.1; visual cylinder length=2 radius=0.1
- link post_link: mass 200 -> 20
Joints:
- joint barrier_joint: limit lower=-3.14 upper=3.14 effort=1000 velocity=10 -> (none); origin xyz=0 0.75 -0.25 rpy=0 0 0 -> xyz=0 0 -0.25 rpy=0 0 0; type revolute -> continuous

File: P1/rampa.urdf (robot description, URDF)
Before this commit: robot ramp, 3 links, 2 joints
Links:
- link base_link: geometry collision box size=2 4 1.5; visual box size=2 4 1.5
- link ramp_left_link: geometry collision box size=2 3.35 0.01; visual box size=2 3.35 0.01
- link ramp_right_link: geometry collision box size=2 3.35 0.01; visual box size=2 3.35 0.01
