Commit message: P1 hecha

File: P1/Mario_Esteban_Practica1/barrera.urdf (robot description, URDF)
Before this commit: robot barrier, 2 links, 1 joints
Links:
- link barrier_link: geometry collision box size=3.0 0.1 0.1; visual box size=3.0 0.1 0.1
- link post_link: mass 20 -> 100; geometry collision cylinder length=1 radius=0.1; visual cylinder length=1 radius=0.15
Joints:
- joint barrier_joint: origin xyz=0 0 -0.25 rpy=0 0 0 -> xyz=0 0 1 rpy=0 0 0

File: P1/Mario_Esteban_Practica1/plataforma.urdf (robot description, URDF)
Before this commit: robot platform, 1 links, 0 joints
Links:
- link platform_link: geometry collision box size=3 1 0.01; visual box size=3 1 0.01
