Commit message: Fase 1 hecha y fase 2 empezada P2

File: P2/rover/urdf/rover.urdf (robot description, URDF)
Before this commit: robot rover, 5 links, 4 joints
Links:
- removed link chasis_link
- added link Chasis_link, mass 12.00000; collision mesh filename=../meshes/dae/Cylinder.001.dae scale=1.00000 1.00000 1.00000; visual mesh filename=../meshes/dae/Cylinder.001.dae scale=1.00000 1.00000 1.00000
- link back_left_wheel_link: mass None -> 2.00000
- link back_right_wheel_link: mass None -> 2.00000
- link front_left_wheel_link: mass None -> 2.00000
- link front_right_wheel_link: mass None -> 2.00000
Joints:
- removed joint front_left_wheel_joint
- added joint front_left_wheel_link_joint: type continuous, parent Chasis_link, child front_left_wheel_link, origin xyz=-1.10001 1.73867 -1.08908 rpy=0.00000 -1.57080 0.00000, axis 0.00000 0.00000 1.00000, limit effort=0.00000 velocity=0.00000
- joint back_left_wheel_link_joint: origin xyz=-1.10000 -1.70000 -1.05020 rpy=0.00000 -1.57080 0.00000 -> xyz=-1.10001 -1.66133 -1.08908 rpy=0.00000 -1.57080 0.00000; parent chasis_link -> Chasis_link
- joint back_right_wheel_link_joint: origin xyz=1.10000 -1.70000 -1.05020 rpy=0.00000 -1.57080 0.00000 -> xyz=1.09999 -1.66133 -1.08908 rpy=0.00000 -1.57080 0.00000; parent chasis_link -> Chasis_link
- joint front_right_wheel_link_joint: origin xyz=1.10000 1.70000 -1.05020 rpy=0.00000 -1.57080 0.00000 -> xyz=1.09999 1.73867 -1.08908 rpy=0.00000 -1.57080 0.00000; parent chasis_link -> Chasis_link

Commit message: Diseño rover terminado

File: P2/rover/urdf/rover.urdf (robot description, URDF)
Before this commit: robot rover, 5 links, 4 joints
Links:
- added link Brazo1_link, mass 1.00000; collision mesh filename=../meshes/dae/Cylinder.dae scale=0.15000 0.50000 0.05000; visual mesh filename=../meshes/dae/Cylinder.dae scale=0.15000 0.50000 0.05000
- added link Brazo2_link, mass 1.50000; collision mesh filename=../meshes/dae/Torus.dae scale=0.18000 0.18000 0.20000; visual mesh filename=../meshes/dae/Torus.dae scale=0.18000 0.18000 0.20000
- added link Brazo3_link, mass 4.00000; collision mesh filename=../meshes/dae/Cylinder.004.dae scale=0.12500 0.12500 1.50000; visual mesh filename=../meshes/dae/Cylinder.004.dae scale=0.12500 0.12500 1.50000
- added link Gripper1_link, mass 0.50000; collision mesh filename=../meshes/dae/Cube.008.dae scale=0.00500 0.12500 0.10000; visual box size=0.01000 0.25000 0.20000
- added link Gripper2_link, mass 0.50000; collision mesh filename=../meshes/dae/Cube.002.dae scale=0.00500 0.12500 0.10000; visual box size=0.01000 0.25000 0.20000
- link Chasis_link: geometry collision mesh filename=../meshes/dae/Cylinder.002.dae scale=0.10000 0.10000 0.50000; visual mesh filename=../meshes/dae/Cylinder.002.dae scale=0.10000 0.10000 0.50000
- link back_left_wheel_link: geometry collision mesh filename=../meshes/dae/Cube.018.dae scale=0.01000 0.01000 0.37500; visual mesh filename=../meshes/dae/Cube.018.dae scale=0.01000 0.01000 0.37500
- link back_right_wheel_link: geometry collision mesh filename=../meshes/dae/Cube.022.dae scale=0.01000 0.01000 0.37500; visual mesh filename=../meshes/dae/Cube.022.dae scale=0.01000 0.01000 0.37500
- link front_left_wheel_link: geometry collision mesh filename=../meshes/dae/Cube.010.dae scale=0.01000 0.01000 0.37500; visual mesh filename=../meshes/dae/Cube.010.dae scale=0.01000 0.01000 0.37500
- link front_right_wheel_link: geometry collision mesh filename=../meshes/dae/Cube.014.dae scale=0.01000 0.01000 0.37500; visual mesh filename=../meshes/dae/Cube.014.dae scale=0.01000 0.01000 0.37500
Joints:
- added joint Brazo1_link_joint: type continuous, parent Chasis_link, child Brazo1_link, origin xyz=-0.00001 0.98058 2.24760 rpy=0.00000 0.00000 0.00000, axis 0.00000 0.00000 1.00000, limit effort=0.00000 velocity=0.00000
- added joint Brazo2_link_joint: type revolute, parent Brazo1_link, child Brazo2_link, origin xyz=-0.00000 0.85000 0.10000 rpy=0.00000 0.00000 0.00000, axis 0.00000 0.00000 1.00000, limit lower=-1.57000 upper=1.57000 effort=0.00000 velocity=0.00000
- added joint Brazo3_link_joint: type prismatic, parent Brazo2_link, child Brazo3_link, origin xyz=-0.00000 1.08500 -2.02499 rpy=0.00000 0.00000 0.00000, axis 0.00000 0.00000 1.00000, limit lower=-0.20000 upper=2.60000 effort=0.00000 velocity=0.00000
- added joint Gripper1_link_joint: type prismatic, parent Brazo3_link, child Gripper1_link, origin xyz=-0.49500 0.00000 -1.04960 rpy=0.00000 0.00000 0.00000, axis 1.00000 0.00000 0.00000, limit lower=0.00000 upper=0.40000 effort=0.00000 velocity=0.00000
- added joint Gripper2_link_joint: type prismatic, parent Brazo3_link, child Gripper2_link, origin xyz=0.49500 0.00000 -1.04960 rpy=0.00000 0.00000 0.00000, axis 1.00000 0.00000 0.00000, limit lower=-0.40000 upper=0.00000 effort=0.00000 velocity=0.00000
- joint back_left_wheel_link_joint: origin xyz=-1.10001 -1.66133 -1.08908 rpy=0.00000 -1.57080 0.00000 -> xyz=-1.10001 -1.66942 -1.10240 rpy=0.00000 -1.57080 0.00000
- joint back_right_wheel_link_joint: origin xyz=1.09999 -1.66133 -1.08908 rpy=0.00000 -1.57080 0.00000 -> xyz=1.09999 -1.66942 -1.10240 rpy=0.00000 -1.57080 0.00000
- joint front_left_wheel_link_joint: origin xyz=-1.10001 1.73867 -1.08908 rpy=0.00000 -1.57080 0.00000 -> xyz=-1.10001 1.73058 -1.10240 rpy=0.00000 -1.57080 0.00000
- joint front_right_wheel_link_joint: origin xyz=1.09999 1.73867 -1.08908 rpy=0.00000 -1.57080 0.00000 -> xyz=1.09999 1.73058 -1.10240 rpy=0.00000 -1.57080 0.00000

Commit message: P2 terminada

File: P2/rover/urdf/rover.urdf (robot description, URDF)
Before this commit: robot rover, 10 links, 9 joints
Links:
- added link Brazo4_link, mass 1.00000; collision mesh filename=../meshes/dae/Cylinder.018.dae scale=0.06875 0.06875 0.88360; visual mesh filename=../meshes/dae/Cylinder.018.dae scale=0.06875 0.06875 0.88360
- added link Brazo5_link, mass 1.00000; collision mesh filename=../meshes/dae/Cube.029.dae scale=0.53959 2.07906 0.16559; visual mesh filename=../meshes/dae/Cube.029.dae scale=0.53959 2.07906 0.16559
- added link Compartimento1_link, mass 1.00000; collision mesh filename=../meshes/dae/Cube.002.dae scale=1.15000 0.00946 0.23944; visual mesh filename=../meshes/dae/Cube.002.dae scale=1.15000 0.00946 0.23944
- added link Compartimento2_link, mass 1.00000; collision mesh filename=../meshes/dae/Cube.003.dae scale=1.15000 0.01000 0.23300; visual mesh filename=../meshes/dae/Cube.003.dae scale=1.15000 0.01000 0.23300
- added link Compartimento3_link, mass 1.00000; collision mesh filename=../meshes/dae/Cube.004.dae scale=0.70000 0.01000 0.23300; visual mesh filename=../meshes/dae/Cube.004.dae scale=0.70000 0.01000 0.23300
- added link Compartimento4_link, mass 1.00000; collision mesh filename=../meshes/dae/Cube.005.dae scale=0.70000 0.01000 0.23300; visual mesh filename=../meshes/dae/Cube.005.dae scale=0.70000 0.01000 0.23300
- link Brazo1_link: mass 1.00000 -> 3.00000; geometry collision mesh filename=../meshes/dae/Cylinder.dae scale=1.00000 0.23300 0.12300; visual mesh filename=../meshes/dae/Cylinder.dae scale=1.00000 0.23300 0.12300
- link Brazo2_link: geometry collision mesh filename=../meshes/dae/Cylinder.013.dae scale=0.67571 0.18837 0.07006; visual mesh filename=../meshes/dae/Cylinder.013.dae scale=0.67571 0.18837 0.07006
- link Brazo3_link: mass 4.00000 -> 1.00000; geometry collision mesh filename=../meshes/dae/Cylinder.016.dae scale=0.09429 0.09429 0.24632; visual mesh filename=../meshes/dae/Cylinder.016.dae scale=0.09429 0.09429 0.24632
- link Chasis_link: mass 12.00000 -> 150.00000; geometry collision mesh filename=../meshes/dae/Cube.dae scale=0.75000 0.37500 0.10000; visual mesh filename=../meshes/dae/Cube.dae scale=0.75000 0.37500 0.10000
- link Gripper1_link: geometry collision mesh filename=../meshes/dae/Cube.031.dae scale=0.53728 0.20000 1.00000; visual mesh filename=../meshes/dae/Cube.031.dae scale=0.53728 0.20000 1.00000
- link Gripper2_link: geometry collision mesh filename=../meshes/dae/Cube.032.dae scale=0.53728 0.20000 1.00000; visual mesh filename=../meshes/dae/Cube.032.dae scale=0.53728 0.20000 1.00000
- link back_left_wheel_link: mass 2.00000 -> 10.00000; geometry collision mesh filename=../meshes/dae/Cube.011.dae scale=0.00500 0.00500 0.22500; visual mesh filename=../meshes/dae/Cube.011.dae scale=0.00500 0.00500 0.22500
- link back_right_wheel_link: mass 2.00000 -> 10.00000; geometry collision mesh filename=../meshes/dae/Cube.013.dae scale=0.00500 0.00500 0.22500; visual mesh filename=../meshes/dae/Cube.013.dae scale=0.00500 0.00500 0.22500
- link front_left_wheel_link: mass 2.00000 -> 10.00000; geometry collision mesh filename=../meshes/dae/Cube.008.dae scale=0.00500 0.00500 0.22500; visual mesh filename=../meshes/dae/Cube.008.dae scale=0.00500 0.00500 0.22500
- link front_right_wheel_link: mass 2.00000 -> 10.00000; geometry collision mesh filename=../meshes/dae/Cube.012.dae scale=0.00500 0.00500 0.22500; visual mesh filename=../meshes/dae/Cube.012.dae scale=0.00500 0.00500 0.22500
Joints:
- added joint Brazo4_link_joint: type prismatic, parent Brazo3_link, child Brazo4_link, origin xyz=-0.00000 -0.00004 -0.14111 rpy=0.00000 0.00000 0.00000, axis 0.00000 0.00000 1.00000, limit lower=-1.50000 upper=0.50000 effort=0.00000 velocity=0.00000
- added joint Brazo5_link_joint: type fixed, parent Brazo4_link, child Brazo5_link, origin xyz=0.00000 0.00000 -0.28645 rpy=0.00000 0.00000 1.57080
- added joint Compartimento1_link_joint: type fixed, parent Chasis_link, child Compartimento1_link, origin xyz=-0.70760 -0.94501 0.24745 rpy=0.00000 0.00000 1.57080
- added joint Compartimento2_link_joint: type fixed, parent Chasis_link, child Compartimento2_link, origin xyz=0.70760 -0.94468 0.24747 rpy=0.00000 0.00000 1.57080
- added joint Compartimento3_link_joint: type fixed, parent Chasis_link, child Compartimento3_link, origin xyz=0.00000 0.17858 0.24745 rpy=0.00000 0.00000 0.00000
- added joint Compartimento4_link_joint: type fixed, parent Chasis_link, child Compartimento4_link, origin xyz=0.00000 -2.06753 0.24745 rpy=0.00000 0.00000 0.00000
- joint Brazo1_link_joint: limit effort=0.00000 velocity=0.00000 -> lower=-3.00000 upper=3.00000 effort=0.00000 velocity=0.00000; origin xyz=-0.00001 0.98058 2.24760 rpy=0.00000 0.00000 0.00000 -> xyz=0.00000 1.05323 1.69829 rpy=0.00000 0.00000 1.57080; type continuous -> revolute
- joint Brazo2_link_joint: limit lower=-1.57000 upper=1.57000 effort=0.00000 velocity=0.00000 -> lower=-2.00000 upper=2.00000 effort=0.00000 velocity=0.00000; origin xyz=-0.00000 0.85000 0.10000 rpy=0.00000 0.00000 0.00000 -> xyz=1.43431 0.00000 0.19480 rpy=0.00000 0.00000 -0.00000
- joint Brazo3_link_joint: limit lower=-0.20000 upper=2.60000 effort=0.00000 velocity=0.00000 -> lower=-1.57000 upper=1.57000 effort=0.00000 velocity=0.00000; origin xyz=-0.00000 1.08500 -2.02499 rpy=0.00000 0.00000 0.00000 -> xyz=1.01188 0.00000 -0.18676 rpy=0.00000 0.00000 -1.57080; type prismatic -> revolute
- joint Gripper1_link_joint: axis 1.00000 0.00000 0.00000 -> 0.00000 0.00000 1.00000; limit lower=0.00000 upper=0.40000 effort=0.00000 velocity=0.00000 -> lower=0.00000 upper=0.30000 effort=0.00000 velocity=0.00000; origin xyz=-0.49500 0.00000 -1.04960 rpy=0.00000 0.00000 0.00000 -> xyz=0.00521 0.50000 -0.28960 rpy=1.57080 1.57080 0.00000; parent Brazo3_link -> Brazo5_link
- joint Gripper2_link_joint: axis 1.00000 0.00000 0.00000 -> 0.00000 0.00000 1.00000; limit lower=-0.40000 upper=0.00000 effort=0.00000 velocity=0.00000 -> lower=-0.30000 upper=0.00000 effort=0.00000 velocity=0.00000; origin xyz=0.49500 0.00000 -1.04960 rpy=0.00000 0.00000 0.00000 -> xyz=0.00520 -0.50000 -0.28960 rpy=1.57080 1.57080 0.00000; parent Brazo3_link -> Brazo5_link
- joint back_left_wheel_link_joint: origin xyz=-1.10001 -1.66942 -1.10240 rpy=0.00000 -1.57080 0.00000 -> xyz=-0.70000 -1.18422 -0.74325 rpy=0.00000 -1.57080 0.00000
- joint back_right_wheel_link_joint: origin xyz=1.09999 -1.66942 -1.10240 rpy=0.00000 -1.57080 0.00000 -> xyz=0.70000 -1.18422 -0.74325 rpy=0.00000 -1.57080 0.00000
- joint front_left_wheel_link_joint: origin xyz=-1.10001 1.73058 -1.10240 rpy=0.00000 -1.57080 0.00000 -> xyz=-0.70000 1.47578 -0.74325 rpy=0.00000 -1.57080 0.00000
- joint front_right_wheel_link_joint: origin xyz=1.09999 1.73058 -1.10240 rpy=0.00000 -1.57080 0.00000 -> xyz=0.70000 1.47578 -0.74325 rpy=0.00000 -1.57080 0.00000
