Commit message: P3 terminada

File: P3/src/rover_description/robots/rover.urdf.xacro (robot description, xacro)
@@ -8,4 +8,5 @@
     <xacro:include filename="$(find rover_description)/urdf/utils/materials.urdf.xacro"/>
     <xacro:include filename="$(find rover_description)/urdf/sensors/sensors.urdf.xacro"/>
+    <xacro:include filename="$(find rover_description)/urdf/ros2_control.urdf.xacro"/>
     <!-- Propiedades -->
     <xacro:property name="PI" value="3.1415926535897931"/>
@@ -13,4 +14,6 @@
     <xacro:arg name="prefix" default=""/>
     <xacro:arg name="robot_ns" default=""/>
+    <xacro:arg name="config_controllers" default="$(find rover_description)/config/rover_controllers.yaml"/>
+    <xacro:arg name="update_rate" default="100"/>
     <!-- Base -->
     <xacro:rover_base prefix="$(arg prefix)"/>
@@ -58,3 +61,5 @@
     <!-- Sensors -->
     <xacro:rover_sensors prefix="$(arg prefix)"/>
+    <!-- Gazebo ROS control plugins -->
+    <xacro:ros2_control/>
 </robot>

File: P3/src/rover_description/urdf/arm/gripper.urdf.xacro (robot description, xacro)
@@ -32,5 +32,5 @@
             <origin rpy="1.57080 1.57080 0.00000" xyz="0.00521 0.50000 -0.28960"/>
             <axis xyz="0.00000 0.00000 1.00000"/>
-            <limit lower="0.00000" upper="0.30000" effort="0.00000" velocity="0.00000"/>
+            <limit lower="0.00000" upper="0.30000" effort="1000" velocity="100.0"/>
         </joint>
         <!-- Gripper 2 -->
@@ -64,6 +64,24 @@
             <origin rpy="1.57080 1.57080 0.00000" xyz="0.00520 -0.50000 -0.28960"/>
             <axis xyz="0.00000 0.00000 1.00000"/>
-            <limit lower="-0.30000" upper="0.00000" effort="0.00000" velocity="0.00000"/>
+            <limit lower="-0.30000" upper="0.00000" effort="1000" velocity="100.0"/>
         </joint>
+        <transmission name="${prefix}Gripper1_link_joint_trans">
+            <type>transmission_interface/SimpleTransmission</type>
+            <joint name="${prefix}Gripper1_link_joint">
+            <hardwareInterface>hardware_interface/PositionJointInterface</hardwareInterface>
+            </joint>
+            <actuator name="${prefix}Gripper1_link_motor">
+            <mechanicalReduction>1</mechanicalReduction>
+            </actuator>
+        </transmission>
+        <transmission name="${prefix}Gripper2_link_joint_trans">
+            <type>transmission_interface/SimpleTransmission</type>
+            <joint name="${prefix}Gripper2_link_joint">
+            <hardwareInterface>hardware_interface/PositionJointInterface</hardwareInterface>
+            </joint>
+            <actuator name="${prefix}Gripper2_link_motor">
+            <mechanicalReduction>1</mechanicalReduction>
+            </actuator>
+        </transmission>
     </xacro:macro>
 </robot>

File: P3/src/rover_description/urdf/arm/scara.urdf.xacro (robot description, xacro)
@@ -32,5 +32,5 @@
             <xacro:insert_block name="origin"/>
             <axis xyz="0.00000 0.00000 1.00000"/>
-            <limit lower="-3.00000" upper="3.00000" effort="0.00000" velocity="0.00000"/>
+            <limit lower="-3.00000" upper="3.00000" effort="1000" velocity="100.0"/>
         </joint>
         <!-- Brazo 2 -->
@@ -64,5 +64,5 @@
             <origin rpy="0.00000 0.00000 0.00000" xyz="1.43431 0.00000 0.19480"/>
             <axis xyz="0.00000 0.00000 1.00000"/>
-            <limit lower="-2.00000" upper="2.00000" effort="0.00000" velocity="0.00000"/>
+            <limit lower="-2.00000" upper="2.00000" effort="1000" velocity="100.0"/>
         </joint>
         <!-- Brazo 3 -->
@@ -96,5 +96,5 @@
             <origin rpy="0.00000 0.00000 -1.57080" xyz="1.01188 0.00000 -0.18676"/>
             <axis xyz="0.00000 0.00000 1.00000"/>
-            <limit lower="-1.57000" upper="1.57000" effort="0.00000" velocity="0.00000"/>
+            <limit lower="-1.57000" upper="1.57000" effort="1000" velocity="100.0"/>
         </joint>
         <!-- Brazo 4 -->
@@ -128,5 +128,5 @@
             <origin rpy="0.00000 0.00000 0.00000" xyz="0.00000 -0.00004 -0.14111"/>
             <axis xyz="0.00000 0.00000 1.00000"/>
-            <limit lower="-1.50000" upper="0.50000" effort="0.00000" velocity="0.00000"/>
+            <limit lower="-1.50000" upper="0.50000" effort="1000" velocity="100.0"/>
         </joint>
         <!-- Brazo 5 -->
@@ -160,4 +160,40 @@
             <origin rpy="0.00000 0.00000 1.57080" xyz="0.00000 0.00000 -0.28645"/>
         </joint>
+        <transmission name="${prefix}Brazo1_link_joint_trans">
+            <type>transmission_interface/SimpleTransmission</type>
+            <joint name="${prefix}Brazo1_link_joint">
+            <hardwareInterface>hardware_interface/PositionJointInterface</hardwareInterface>
+            </joint>
+            <actuator name="${prefix}Brazo1_link_motor">
+            <mechanicalReduction>1</mechanicalReduction>
+            </actuator>
+        </transmission>
+        <transmission name="${prefix}Brazo2_link_joint_trans">
+            <type>transmission_interface/SimpleTransmission</type>
+            <joint name="${prefix}Brazo2_link_joint">
+            <hardwareInterface>hardware_interface/PositionJointInterface</hardwareInterface>
+            </joint>
+            <actuator name="${prefix}Brazo2_link_motor">
+            <mechanicalReduction>1</mechanicalReduction>
+            </actuator>
+        </transmission>
+        <transmission name="${prefix}Brazo3_link_joint_trans">
+            <type>transmission_interface/SimpleTransmission</type>
+            <joint name="${prefix}Brazo3_link_joint">
+            <hardwareInterface>hardware_interface/PositionJointInterface</hardwareInterface>
+            </joint>
+            <actuator name="${prefix}Brazo3_link_motor">
+            <mechanicalReduction>1</mechanicalReduction>
+            </actuator>
+        </transmission>
+        <transmission name="${prefix}Brazo4_link_joint_trans">
+            <type>transmission_interface/SimpleTransmission</type>
+            <joint name="${prefix}Brazo4_link_joint">
+            <hardwareInterface>hardware_interface/PositionJointInterface</hardwareInterface>
+            </joint>
+            <actuator name="${prefix}Brazo4_link_motor">
+            <mechanicalReduction>1</mechanicalReduction>
+            </actuator>
+        </transmission>
     </xacro:macro>
 </robot>

File: P3/src/rover_description/urdf/wheels/rover_wheel.urdf.xacro (robot description, xacro)
@@ -30,6 +30,19 @@
       <origin xyz="${joint_xyz}" rpy="${joint_rpy}"/>
       <axis xyz="0 0 1"/>
-      <limit effort="0.0" velocity="0.0"/>
+      <limit effort="1000.0" velocity="100.0"/>
     </joint>
+    <transmission name="${prefix}wheel_link_joint_trans">
+      <type>transmission_interface/SimpleTransmission</type>
+      <joint name="${prefix}wheel_link_joint">
+        <hardwareInterface>hardware_interface/VelocityJointInterface</hardwareInterface>
+      </joint>
+      <actuator name="${prefix}wheel_link_motor">
+        <mechanicalReduction>1</mechanicalReduction>
+      </actuator>
+    </transmission>
+<gazebo reference="${prefix}wheel_link">
+  <mu1>5</mu1>
+  <mu2>5</mu2>
+</gazebo>
   </xacro:macro>
 </robot>
